File: kicad/nabu_led_pcb/nabu_led_pcb.kicad_sch (KiCad schematic)
At the start: 6 parts, among them P1 Conn_01x06_Pin

Commit message: Updated to latest KiCAD.
Other:
- title: NABU PC Front Panel Board -> NABU PC Front Panel LED Board
Changed lines of the file:
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@@
   (paper "A4")
   (title_block
-    (title "NABU PC Front Panel Board")
+    (title "NABU PC Front Panel LED Board")
     (date "June 12, 2023")
     (rev "A")
@@
     (data
       iVBORw0KGgoAAAANSUhEUgAAAloAAACaCAIAAAD+TnEgAAAAA3NCSVQICAjb4U/gAAAACXBIWXMA
-      AAsSAAALEgHS3X78AAAgAElEQVR4nHS9WbMkS24mhsXdIyIzz1bL3auHbJItzpPmiX9GMtNQ4pA0
+      AArwAAAK8AFCrDSYAAAgAElEQVR4nHS9WbMkS24mhsXdIyIzz1bL3auHbJItzpPmiX9GMtNQ4pA0
       cmb0L2WmF73qSTYku4fdfe+tqrNkRoQvAPSADD9Rl1LasbJTJyMj3OFw4MMHwBN/90//9+VyqbWm
       lMZxVNV1XWutzNxaExFmJiJEJCJiFrEizcxCCCklM8vbK6UUQvArmdnMas0iEqP/XrU1ZmZmACBA
@@
     )
   )
-  (image (at 82.55 124.46) (scale 2.54394)
+  (image (at 81.28 123.19) (scale 2.54394)
     (data
       iVBORw0KGgoAAAANSUhEUgAAAk4AAADnCAIAAABnt06tAAAAA3NCSVQICAjb4U/gAAAACXBIWXMA
-      AAsSAAALEgHS3X78AAAgAElEQVR4nLS9abPkym0gCiCTZG3nnN5u910k2fK8ePEiHP7/P8KfxuGY
+      AArwAAAK8AFCrDSYAAAgAElEQVR4nLS9abPkym0gCiCTZG3nnN5u910k2fK8ePEiHP7/P8KfxuGY
       GVuyLEu6Sy9nq51kJvA+gESByTotTcQMo+N0FYvMRGJPJBKJ//5v/wovXyJinxHxK/f9nctn5MAg
       kPUmQkBEIETEPou+i4iCKCLMLCKBLw0ysz5DRDhe2rA+LMBEBMDao/UrIjFGe16bYmbmFAQQxTeY
